File: Kicad/Regulador de voltaje con proteccion de diodos/Proyect1_RDVCPDD/Proyect1_RDVCPDD.kicad_sch (KiCad schematic)
At the start: 11 parts, among them J1 Screw_Terminal_01x02, J2 Screw_Terminal_01x02

Commit message: [UPDATE] Kicad *
Parts:
- C1: footprint (none) -> Capacitor_SMD:C_0603_1608Metric
- C2, C3: footprint (none) -> Capacitor_SMD:CP_Elec_6.3x5.8
- D1, D2, D3: footprint (none) -> Diode_SMD:D_SMA
- J1, J2: footprint (none) -> TerminalBlock_Phoenix:TerminalBlock_Phoenix_MKDS-1,5-2-5.08_1x02_P5.08mm_Horizontal
- R1: footprint (none) -> Resistor_SMD:R_1206_3216Metric
- RV1: footprint (none) -> Potentiometer_THT:Potentiometer_Bourns_3296W_Vertical
- gave numbers to parts that had none: 1
Changed lines of the file:
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@@
     (effects (font (size 3 3) (thickness 0.254) bold) (justify left bottom))
+  )
+  (symbol (lib_id "Device:C_Polarized") (at 132.08 55.88 0) (unit 1)
+    (in_bom yes) (on_board yes)
+    (property "Reference" "C3" (id 0) (at 135.89 53.7209 0)
+      (effects (font (size 1.27 1.27)) (justify left))
+    )
+    (property "Value" "C_Polarized" (id 1) (at 135.89 56.2609 0)
+      (effects (font (size 1.27 1.27)) (justify left) hide)
+    )
+    (property "Footprint" "Capacitor_SMD:CP_Elec_6.3x5.8" (id 2) (at 133.0452 59.69 0)
+      (effects (font (size 1.27 1.27)) hide)
+    )
+    (property "Datasheet" "~" (id 3) (at 132.08 55.88 0)
+      (effects (font (size 1.27 1.27)) hide)
+    )
+    (pin "1")
+    (pin "2")
   )
   (symbol (lib_id "Simulation_SPICE:DIODE") (at 78.74 49.53 0) (unit 1)
@@
       (effects (font (size 1.27 1.27)) hide)
     )
-    (property "Footprint" "" (id 2) (at 78.74 49.53 0)
+    (property "Footprint" "Diode_SMD:D_SMA" (id 2) (at 78.74 49.53 0)
       (effects (font (size 1.27 1.27)) hide)
     )
@@
       (effects (font (size 1.27 1.27)) hide)
     )
-    (property "Footprint" "" (id 2) (at 68.58 52.07 0)
+    (property "Footprint" "TerminalBlock_Phoenix:TerminalBlock_Phoenix_MKDS-1,5-2-5.08_1x02_P5.08mm_Horizontal" (id 2) (at 68.58 52.07 0)
       (effects (font (size 1.27 1.27)) hide)
     )
@@
       (effects (font (size 1.27 1.27)) (justify right) hide)
     )
-    (property "Footprint" "" (id 2) (at 109.22 55.88 0)
+    (property "Footprint" "Diode_SMD:D_SMA" (id 2) (at 109.22 55.88 0)
       (effects (font (size 1.27 1.27)) hide)
     )
@@
   (symbol (lib_id "Regulator_Linear:LM317_TO-252") (at 96.52 49.53 0) (unit 1)
     (in_bom yes) (on_board yes) (fields_autoplaced)
-    (property "Reference" "U?" (id 0) (at 96.52 41.91 0))
+    (property "Reference" "U1" (id 0) (at 96.52 41.91 0))
     (property "Value" "LM317_TO-252" (id 1) (at 96.52 44.45 0))
     (property "Footprint" "Package_TO_SOT_SMD:TO-252-2" (id 2) (at 96.52 43.18 0)
@@
   (symbol (lib_id "power:GND") (at 96.52 81.28 0) (unit 1)
     (in_bom yes) (on_board yes) (fields_autoplaced)
-    (property "Reference" "#PWR?" (id 0) (at 96.52 87.63 0)
+    (property "Reference" "#PWR0101" (id 0) (at 96.52 87.63 0)
       (effects (font (size 1.27 1.27)) hide)
     )
@@
       (effects (font (size 1.27 1.27)) (justify right) hide)
     )
-    (property "Footprint" "" (id 2) (at 96.52 69.85 0)
+    (property "Footprint" "Potentiometer_THT:Potentiometer_Bourns_3296W_Vertical" (id 2) (at 96.52 69.85 0)
       (effects (font (size 1.27 1.27)) hide)
     )
@@
       (effects (font (size 1.27 1.27)) (justify left) hide)
     )
-    (property "Footprint" "" (id 2) (at 110.1852 73.66 0)
+    (property "Footprint" "Capacitor_SMD:CP_Elec_6.3x5.8" (id 2) (at 110.1852 73.66 0)
       (effects (font (size 1.27 1.27)) hide)
     )
@@
     (pin "2")
   )
-  (symbol (lib_id "Device:C_Polarized") (at 132.08 55.88 0) (unit 1)
-    (in_bom yes) (on_board yes) (fields_autoplaced)
-    (property "Reference" "C3" (id 0) (at 135.89 54.9909 0)
-      (effects (font (size 1.27 1.27)) (justify left))
-    )
-    (property "Value" "C_Polarized" (id 1) (at 135.89 56.2609 0)
-      (effects (font (size 1.27 1.27)) (justify left) hide)
-    )
-    (property "Footprint" "" (id 2) (at 133.0452 59.69 0)
-      (effects (font (size 1.27 1.27)) hide)
-    )
-    (property "Datasheet" "~" (id 3) (at 132.08 55.88 0)
-      (effects (font (size 1.27 1.27)) hide)
-    )
-    (pin "1")
-    (pin "2")
-  )
   (symbol (lib_id "Device:R_US") (at 120.65 55.88 0) (unit 1)
     (in_bom yes) (on_board yes) (fields_autoplaced)
@@
     )
     (property "Value" "R_US" (id 1) (at 123.19 57.1499 0)
-      (effects (font (size 1.27 1.27)) (justify left) hide)
-    )
-    (property "Footprint" "" (id 2) (at 121.666 56.134 90)
+      (effects (font (size 1.27 1.27)) (justify left))
+    )
+    (property "Footprint" "Resistor_SMD:R_1206_3216Metric" (id 2) (at 121.666 56.134 90)
       (effects (font (size 1.27 1.27)) hide)
     )
@@
       (effects (font (size 1.27 1.27)) (justify left) hide)
     )
-    (property "Footprint" "" (id 2) (at 86.0552 63.5 0)
+    (property "Footprint" "Capacitor_SMD:C_0603_1608Metric" (id 2) (at 86.0552 63.5 0)
       (effects (font (size 1.27 1.27)) hide)
     )
@@
       (effects (font (size 1.27 1.27)) hide)
     )
-    (property "Footprint" "" (id 2) (at 99.06 39.37 0)
+    (property "Footprint" "Diode_SMD:D_SMA" (id 2) (at 99.06 39.37 0)
       (effects (font (size 1.27 1.27)) hide)
     )
@@
       (effects (font (size 1.27 1.27)) (justify left) hide)
     )
-    (property "Footprint" "" (id 2) (at 144.78 49.53 0)
+    (property "Footprint" "TerminalBlock_Phoenix:TerminalBlock_Phoenix_MKDS-1,5-2-5.08_1x02_P5.08mm_Horizontal" (id 2) (at 144.78 49.53 0)
       (effects (font (size 1.27 1.27)) hide)
     )
@@
   (symbol_instances
     (path "/61b0a90c-0888-4889-b915-b5a54dbc418f"
-      (reference "#PWR?") (unit 1) (value "GND") (footprint "")
+      (reference "#PWR0101") (unit 1) (value "GND") (footprint "")
     )
     (path "/b0125b25-42ba-45e1-8d55-f8d94e2e07a0"
-      (reference "C1") (unit 1) (value "C") (footprint "")
+      (reference "C1") (unit 1) (value "C") (footprint "Capacitor_SMD:C_0603_1608Metric")
     )
     (path "/9558250b-c2b1-4d7d-84b8-5d33c93cea18"
-      (reference "C2") (unit 1) (value "C_Polarized") (footprint "")
-    )
-    (path "/99063065-2d13-4b41-a0c6-32e0677cf1e3"
-      (reference "C3") (unit 1) (value "C_Polarized") (footprint "")
+      (reference "C2") (unit 1) (value "C_Polarized") (footprint "Capacitor_SMD:CP_Elec_6.3x5.8")
+    )
+    (path "/0c19dbaa-13be-4ae3-b406-b227cbf2821a"
+      (reference "C3") (unit 1) (value "C_Polarized") (footprint "Capacitor_SMD:CP_Elec_6.3x5.8")
     )
     (path "/3b47b150-9d13-415f-a5aa-e67c705042a3"
-      (reference "D1") (unit 1) (value "DIODE") (footprint "")
+      (reference "D1") (unit 1) (value "DIODE") (footprint "Diode_SMD:D_SMA")
     )
     (path "/c231bb92-7ab6-49f8-8500-237f9e5edfc5"
-      (reference "D2") (unit 1) (value "DIODE") (footprint "")
+      (reference "D2") (unit 1) (value "DIODE") (footprint "Diode_SMD:D_SMA")
     )
     (path "/0c6ec339-9ef0-43e1-8d08-69c39af74f96"
-      (reference "D3") (unit 1) (value "DIODE") (footprint "")
+      (reference "D3") (unit 1) (value "DIODE") (footprint "Diode_SMD:D_SMA")
     )
     (path "/2a77b02a-4cd0-455b-8422-3eb8919ac7d7"
-      (reference "J1") (unit 1) (value "Screw_Terminal_01x02") (footprint "")
+      (reference "J1") (unit 1) (value "Screw_Terminal_01x02") (footprint "TerminalBlock_Phoenix:TerminalBlock_Phoenix_MKDS-1,5-2-5.08_1x02_P5.08mm_Horizontal")
     )
     (path "/df396970-03d2-4c41-b642-05f45f8c01d6"
-      (reference "J2") (unit 1) (value "Screw_Terminal_01x02") (footprint "")
+      (reference "J2") (unit 1) (value "Screw_Terminal_01x02") (footprint "TerminalBlock_Phoenix:TerminalBlock_Phoenix_MKDS-1,5-2-5.08_1x02_P5.08mm_Horizontal")
     )
     (path "/adac5a1e-a51a-4d13-85c1-292163991bc5"
-      (reference "R1") (unit 1) (value "R_US") (footprint "")
+      (reference "R1") (unit 1) (value "R_US") (footprint "Resistor_SMD:R_1206_3216Metric")
     )
     (path "/70dc3af9-e335-4852-842c-bdd6dfe00046"
-      (reference "RV1") (unit 1) (value "R_Potentiometer_Trim_US") (footprint "")
+      (reference "RV1") (unit 1) (value "R_Potentiometer_Trim_US") (footprint "Potentiometer_THT:Potentiometer_Bourns_3296W_Vertical")
     )
     (path "/43cf5d99-3bf8-401d-8b25-7b30b91e22ed"
-      (reference "U?") (unit 1) (value "LM317_TO-252") (footprint "Package_TO_SOT_SMD:TO-252-2")
-    )
-  )
+      (reference "U1") (unit 1) (value "LM317_TO-252") (footprint "Package_TO_SOT_SMD:TO-252-2")
+    )
+  )
