File: Kicad/Regulador de voltaje con proteccion de diodos/Proyect1_RDVCPDD/Proyect1_RDVCPDD.kicad_pcb (KiCad board)
At the start: 2 copper layers, 50 x 30 mm, 4 parts

Commit message: [UPDATE] Kicad *
Parts:
- added C1: C, Capacitor_SMD:C_0603_1608Metric, F.Cu at (1054.0, -143.0)
- added C2: C_Polarized, Capacitor_SMD:CP_Elec_6.3x5.8, F.Cu at (1072.0, -146.7)
- added C3: C_Polarized, Capacitor_SMD:CP_Elec_6.3x5.8, F.Cu at (1072.0, -158.0)
- added D1: DIODE, Diode_SMD:D_SMA, F.Cu at (1056.0, -161.0)
- added D2: DIODE, Diode_SMD:D_SMA, F.Cu at (1064.0, -161.0)
- added D3: DIODE, Diode_SMD:D_SMA, F.Cu at (1056.0, -147.0)
- added J1: Screw_Terminal_01x02, TerminalBlock_Phoenix:TerminalBlock_Phoenix_MKDS-1,5-2-5.08_1x02_P5.08mm_Horizontal, F.Cu at (1046.0, -157.5)
- added J2: Screw_Terminal_01x02, TerminalBlock_Phoenix:TerminalBlock_Phoenix_MKDS-1,5-2-5.08_1x02_P5.08mm_Horizontal, F.Cu at (1084.0, -152.5)
- added R1: R_US, Resistor_SMD:R_1206_3216Metric, F.Cu at (1064.0, -165.0)
- added RV1: R_Potentiometer_Trim_US, Potentiometer_THT:Potentiometer_Bourns_3296W_Vertical, F.Cu at (1076.0, -166.0)
- added U1: LM317_TO-252, Package_TO_SOT_SMD:TO-252-2, F.Cu at (1058.2, -154.5)

Commit message: [UPDATE] Kicad/Pr1 *
Routing:
- net GND: track 0.00 -> 75.9 mm, vias 0 -> 2
- net Net-(C3-Pad1): track 0.00 -> 67.6 mm
- net Net-(C2-Pad1): track 0.00 -> 55.1 mm, vias 0 -> 2
- net Net-(C1-Pad1): track 0.00 -> 35.1 mm
- net Net-(D3-Pad1): track 0.00 -> 12.3 mm
- added copper zone on F.Cu, net (none)
